File: SPECTRE_V0.6/Speeduino_base.sch (KiCad schematic (older format))
At the start: 234 parts, among them J1 Conn_01x06_Male, J2 Conn_02x04_Odd_Even, Q1 2N7002, Q10 AO3401A, Q11 AO3401A, Q12 BSP78, Q13 BSP78, Q14 BSP78, Q15 BSP78, Q16 BSP78, Q17 SMD-MOSFET-N-CH-55V-2.1A-AO34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, Q18 BSP78, Q19 SMD-MOSFET-N-CH-55V-2.1A-AO34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, Q2 CJ2302, Q20 AO3401A, Q21 BSP78, Q22 AO3401A, Q23 BSP78, Q24 BSP78, Q25 BSP78, Q26 BSP78, Q3 CJ2302, Q4 CJ2302, Q5 CJ2302, Q6 CJ2302, Q7 CJ2302, Q8 SMD-MOSFET-N-CH-55V-2.1A-AO34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, Q9 SMD-MOSFET-N-CH-55V-2.1A-AO34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, U1 MAX9926UAEE+, U10 74LS08, U11 74LS08, U12 TJA1050, U14 MAX3232, U2 LM78M05_TO220, U3 TL431DBZ, U4 74LS32, U5 molex_48pin, U6 LM2901, U7 LTC6992, U8 74LS74, U9 74LS74

Commit message: Cleaned and updated the SPECTRE V0.5 Created separate Peak and Hold board.
Parts:
- D18, D22: value SS310 -> LL4148; footprint Diode_SMD:D_SOD-123 -> Diode_SMD:D_MiniMELF
Changed lines of the file:
@@
 P 6350 2100
 F 0 "D18" H 6350 1987 50  0000 C CNN
-F 1 "SS310" V 6395 2168 50  0001 L CNN
-F 2 "Diode_SMD:D_SOD-123" V 6350 2100 50  0001 C CNN
+F 1 "LL4148" V 6395 2168 50  0001 L CNN
+F 2 "Diode_SMD:D_MiniMELF" V 6350 2100 50  0001 C CNN
 F 3 "~" V 6350 2100 50  0001 C CNN
 	1    6350 2100
@@
 P 8450 2300
 F 0 "D22" H 8450 2187 50  0000 C CNN
-F 1 "SS310" V 8495 2368 50  0001 L CNN
-F 2 "Diode_SMD:D_SOD-123" V 8450 2300 50  0001 C CNN
+F 1 "LL4148" V 8495 2368 50  0001 L CNN
+F 2 "Diode_SMD:D_MiniMELF" V 8450 2300 50  0001 C CNN
 F 3 "~" V 8450 2300 50  0001 C CNN
 	1    8450 2300
