File: SPECTRE_V0.5.2/Speeduino_base.sch (KiCad schematic (older format))
At the start: 211 parts, among them J1 Conn_01x06_Male, J2 Conn_02x04_Odd_Even, J3 ProtoArea, Q1 AO3400, Q10 BSP78, Q11 BSP78, Q12 AO3400, Q13 BSP78, Q14 BSP78, Q15 BSP78, Q16 BSP78, Q17 BSP78, Q18 BSP78, Q19 BSP78, Q20 BSP78, Q21 BSP78, Q6 AO3400, Q7 AO3400, U1 MAX9926UAEE+, U10 MIC4427, U2 LM78M05_TO220, U3 TL431DBZ, U4 molex_48pin, U5 TJA1050, U6 MAX3232, U7 MIC4427, U8 MIC4427, U9 MIC4427

Commit message: update molex 48 pin to correct location
Parts:
- removed U4: molex_48pin, rusefi_lib:Molex_48, symbol molex_48pin:molex_48pin
- added U4: molex_48pin, Speeduino_base:Molex_48, symbol speeduino_lib:molex_48pin
- U2: footprint Package_TO_SOT_THT:TO-220-3_Horizontal_TabUp -> Package_TO_SOT_THT:TO-220-3_Vertical
Connections:
- net 3.3V: now also U4.46
- net 5V: now also U4.37
- net AIN_1: now also U4.18
- net AIN_2: now also U4.14
- net AIN_3: now also U4.20
- net BARO: now also U4.10
- net BOOST-OUT: now also U4.47
- net CANH: now also U4.29
- net CANL: now also U4.45
- net CLT: now also U4.27
- net FAN: now also U4.15
- net FLEX_FUEL_IN: now also U4.38
- net FUEL_PUMP: now also U4.19
- net GND: now also U4.30, U4.33
- net IAT: now also U4.17
- net IGN1-OUT: now also U4.13
- net IGN2-OUT: now also U4.31
- net IGN3-OUT: now also U4.36
- net IGN4-OUT: now also U4.40
- net INJ1-OUT: now also U4.32
- net INJ2-OUT: now also U4.44
- net INJ3-OUT: now also U4.28
- net INJ4-OUT: now also U4.24
- net INJ5-OUT: now also U4.7
- net INJ6-OUT: now also U4.8
- net INJ7-OUT: now also U4.6
- net INJ8-OUT: now also U4.5
- net MAP: now also U4.25
- net O2: now also U4.23
- net PWR_GND: now also U4.1, U4.2
- net RS232_RX: now also U4.34
- net RS232_TX: now also U4.21
- net TACHO-OUT: now also U4.48
- net TPS: now also U4.35
- net VBAT: now also U4.3, U4.4
- net VR1+: now also U4.43
- net VR1-: now also U4.42
- net VR2+: now also U4.41
- net VR2-: now also U4.39
- net at JP6.2 (C): now also U4.11
- net at JP7.2 (C): now also U4.12
- net at JP8.2 (C): now also U4.16
- net at JP18.2 (C): now also U4.22
- net at JP16.2 (C): now also U4.26
- net at JP5.2 (C): now also U4.9
Changed lines of the file:
@@
 Wire Wire Line
 	4000 1400 3950 1400
-Wire Wire Line
-	4100 1400 4200 1400
 Text GLabel 3950 1850 3    50   Output ~ 0
 PWR_GND
@@
 F 0 "U2" H 2700 11042 50  0000 C CNN
 F 1 "LM78M05_TO220" H 2700 10951 50  0000 C CNN
-F 2 "Package_TO_SOT_THT:TO-220-3_Horizontal_TabUp" H 2700 11025 50  0001 C CIN
+F 2 "Package_TO_SOT_THT:TO-220-3_Vertical" H 2700 11025 50  0001 C CIN
 F 3 "http://www.fairchildsemi.com/ds/LM/LM78M05.pdf" H 2700 10750 50  0001 C CNN
 	1    2700 10800
@@
 Text GLabel 6100 1400 3    50   Input ~ 0
 RS232_TX
-Connection ~ 4200 1400
-$Comp
-L molex_48pin:molex_48pin U4
-U 1 1 5E17AB54
-P 6900 1950
-F 0 "U4" V 8187 2355 60  0000 C CNN
-F 1 "molex_48pin" V 8081 2355 60  0000 C CNN
-F 2 "rusefi_lib:Molex_48" H 6900 1950 60  0001 C CNN
-F 3 "" H 6900 1950 60  0001 C CNN
-	1    6900 1950
-	0    -1   -1   0
-$EndComp
 Text GLabel 7500 1400 3    50   Output ~ 0
 RS232_RX
@@
 Wire Wire Line
 	12150 9150 12200 9150
+Wire Wire Line
+	4100 1400 4200 1400
+$Comp
+L speeduino_lib:molex_48pin U4
+U 1 1 60019D12
+P 6900 1950
+F 0 "U4" V 8187 2355 60  0000 C CNN
+F 1 "molex_48pin" V 8081 2355 60  0000 C CNN
+F 2 "Speeduino_base:Molex_48" H 6900 1950 60  0001 C CNN
+F 3 "" H 6900 1950 60  0001 C CNN
+	1    6900 1950
+	0    -1   -1   0
+$EndComp
+Connection ~ 4200 1400
 $EndSCHEMATC
