File: SPECTRE_V0.5.3/Speeduino_base.sch (KiCad schematic (older format))
At the start: 217 parts, among them J1 Conn_01x06_Male, J2 Conn_02x04_Odd_Even, J3 ProtoArea, Q1 AO3400, Q10 BSP78, Q11 BSP78, Q12 AO3400, Q13 BSP78, Q14 BSP78, Q15 BSP78, Q16 BSP78, Q17 BSP78, Q18 BSP78, Q19 BSP78, Q20 BSP78, Q21 BSP78, Q6 AO3400, Q7 AO3400, U1 MAX9926UAEE+, U10 MIC4427, U2 LM78M05_TO220, U3 TL431DBZ, U4 molex_48pin, U5 TJA1050, U6 MAX3232, U7 MIC4427, U8 MIC4427, U9 MIC4427

Commit message: Update V0.5.3 Update JLCpcb part numbers in schematic Updated board layout. Added bom for JLCPCB SMT service Added location file for JLCPCB SMT service
Parts:
- C11: LCSC (none) -> C21120
- C12, C18: LCSC (none) -> C250105
- C15: LCSC (none) -> C13585
- C30: LCSC (none) -> C14663
- C5, C7: LCSC (none) -> C1588
- D22: LCSC (none) -> C19726
- D28: LCSC (none) -> C72038
- D32: LCSC (none) -> C110856
- F1, F2: LCSC (none) -> C70122
- Q1: LCSC (none) -> C344010
- R20: LCSC (none) -> C21189
- R22, R31: LCSC (none) -> C126158
- R23: LCSC (none) -> C23179
- R25: LCSC (none) -> C23162
- R26: LCSC (none) -> C23260
- R30, R35: LCSC (none) -> C21190
- R40: LCSC (none) -> C22775
- R44: LCSC (none) -> C4216
- R45: LCSC (none) -> C23186
- R70: LCSC Part # (none) -> C22859
- R71: LCSC (none) -> C22859
- R74: LCSC (none) -> C22787
- R75: LCSC (none) -> C22962
- R90: LCSC (none) -> C25803
- U10, U7, U8, U9: LCSC (none) -> C49058
- U5: LCSC (none) -> C6952
Changed lines of the file:
@@
 $EndComp
 $Comp
-L Speeduino_base-eagle-import:CERAMIC-10UF-25V-10%-X5R(1206) C15
-U 1 1 603F19F2
-P 3250 1090
-F 0 "C15" H 3100 1140 42  0000 L BNN
-F 1 "10uf" H 3100 990 42  0000 L BNN
-F 2 "Speeduino_base:C1206" H 3250 1090 50  0001 C CNN
-F 3 "" H 3250 1090 50  0001 C CNN
-	1    3250 1090
-	0    -1   -1   0
-$EndComp
-$Comp
 L Speeduino_base-eagle-import:MAX9926UAEE+ U1
 U 1 1 F9562130
@@
 F 2 "Speeduino_base:C0603" H 8500 10850 50  0001 C CNN
 F 3 "" H 8500 10850 50  0001 C CNN
+F 4 "C1588" H 8500 10850 50  0001 C CNN "LCSC"
 	1    8500 10850
 	-1   0    0    1
@@
 F 2 "Speeduino_base:C0603" H 9000 10850 50  0001 C CNN
 F 3 "" H 9000 10850 50  0001 C CNN
+F 4 "C1588" H 9000 10850 50  0001 C CNN "LCSC"
 	1    9000 10850
 	-1   0    0    1
@@
 F 2 "Speeduino_base:R0603" H 3650 7800 50  0001 C CNN
 F 3 "" H 3650 7800 50  0001 C CNN
+F 4 "C21190" H 3650 7800 50  0001 C CNN "LCSC"
 	1    3650 7800
 	-1   0    0    1
@@
 F 2 "Resistor_SMD:R_1812_4532Metric_Pad1.30x3.40mm_HandSolder" H 1200 950 50  0001 C CNN
 F 3 "" H 1200 950 50  0001 C CNN
+F 4 "C70122" H 1200 950 50  0001 C CNN "LCSC"
 	1    1200 950
 	-1   0    0    1
@@
 F 2 "Speeduino_base:LED-0603" H 11650 4150 50  0001 C CNN
 F 3 "" H 11650 4150 50  0001 C CNN
+F 4 "C72038" H 11650 4150 50  0001 C CNN "LCSC"
 	1    11650 4150
 	1    0    0    -1
@@
 F 2 "Speeduino_base:R0603" H 11150 3350 50  0001 C CNN
 F 3 "" H 11150 3350 50  0001 C CNN
+F 4 "C22962" H 11150 3350 50  0001 C CNN "LCSC"
 	1    11150 3350
 	-1   0    0    1
@@
 F 2 "Speeduino_base:R0603" H 2500 1600 50  0001 C CNN
 F 3 "" H 2500 1600 50  0001 C CNN
+F 4 "C21189" H 2500 1600 50  0001 C CNN "LCSC"
 	1    2500 1600
 	1    0    0    -1
@@
 	3550 1300 3850 1300
 Wire Wire Line
-	3250 900  3250 940
-Connection ~ 3250 940
-Wire Wire Line
-	3250 940  3250 950
-Wire Wire Line
-	3550 900  3250 900
-Connection ~ 3250 900
-Wire Wire Line
 	3850 950  3850 900
 Wire Wire Line
@@
 Wire Wire Line
 	2300 900  2500 900
-Wire Wire Line
-	3100 900  3250 900
 Text GLabel 7000 1250 3    50   Input ~ 0
 INJ6-OUT
@@
 F 2 "Resistor_SMD:R_1812_4532Metric_Pad1.30x3.40mm_HandSolder" H 1250 1650 50  0001 C CNN
 F 3 "" H 1250 1650 50  0001 C CNN
+F 4 "C70122" H 1250 1650 50  0001 C CNN "LCSC"
 	1    1250 1650
 	-1   0    0    1
@@
 F 2 "Package_SO:SO-8_5.3x6.2mm_P1.27mm" H 13800 7900 50  0001 C CNN
 F 3 "" H 13800 7900 50  0001 C CNN
+F 4 "C6952" H 13800 7900 50  0001 C CNN "LCSC"
 	1    13800 7900
 	1    0    0    -1
@@
 F 2 "Speeduino_base:C0603" H 12850 10450 50  0001 C CNN
 F 3 "~" H 12850 10450 50  0001 C CNN
+F 4 "C14663" H 12850 10450 50  0001 C CNN "LCSC"
 	1    12850 10450
 	0    1    1    0
@@
 F 2 "Speeduino_base:R0603" H 14400 7800 50  0001 C CNN
 F 3 "" H 14400 7800 50  0001 C CNN
+F 4 "C22787" H 14400 7800 50  0001 C CNN "LCSC"
 	1    14400 7800
 	0    -1   -1   0
@@
 F 2 "Speeduino_base:R0603" H 3050 1950 50  0001 C CNN
 F 3 "~" H 3050 1950 50  0001 C CNN
+F 4 "C21190" H 3050 1950 50  0001 C CNN "LCSC"
 	1    3050 1950
 	1    0    0    -1
@@
 F 2 "Speeduino_base:R0603" H 3050 2250 50  0001 C CNN
 F 3 "~" H 3050 2250 50  0001 C CNN
+F 4 "C126158" H 3050 2250 50  0001 C CNN "LCSC"
 	1    3050 2250
 	1    0    0    -1
@@
 F 2 "Capacitor_SMD:CP_Elec_6.3x7.7" H 2600 2100 50  0001 C CNN
 F 3 "~" H 2600 2100 50  0001 C CNN
+F 4 "C250105" H 2600 2100 50  0001 C CNN "LCSC"
 	1    2600 2100
 	1    0    0    -1
@@
 F 2 "Capacitor_SMD:CP_Elec_6.3x7.7" H 4150 1100 50  0001 C CNN
 F 3 "~" H 4150 1100 50  0001 C CNN
+F 4 "C250105" H 4150 1100 50  0001 C CNN "LCSC"
 	1    4150 1100
 	1    0    0    -1
@@
 F 2 "Package_SO:SO-8_3.9x4.9mm_P1.27mm" H 600 6200 50  0001 C CNN
 F 3 "http://ww1.microchip.com/downloads/en/DeviceDoc/mic4426.pdf" H 600 6200 50  0001 C CNN
+F 4 "C49058" H 600 6500 50  0001 C CNN "LCSC"
 	1    600  6500
 	1    0    0    -1
@@
 F 2 "Package_SO:SO-8_3.9x4.9mm_P1.27mm" H 2200 6200 50  0001 C CNN
 F 3 "http://ww1.microchip.com/downloads/en/DeviceDoc/mic4426.pdf" H 2200 6200 50  0001 C CNN
+F 4 "C49058" H 2200 6500 50  0001 C CNN "LCSC"
 	1    2200 6500
 	1    0    0    -1
@@
 F 2 "Package_SO:SO-8_3.9x4.9mm_P1.27mm" H 3900 6200 50  0001 C CNN
 F 3 "http://ww1.microchip.com/downloads/en/DeviceDoc/mic4426.pdf" H 3900 6200 50  0001 C CNN
+F 4 "C49058" H 3900 6500 50  0001 C CNN "LCSC"
 	1    3900 6500
 	1    0    0    -1
@@
 F 2 "Package_SO:SO-8_3.9x4.9mm_P1.27mm" H 5950 6200 50  0001 C CNN
 F 3 "http://ww1.microchip.com/downloads/en/DeviceDoc/mic4426.pdf" H 5950 6200 50  0001 C CNN
+F 4 "C49058" H 5950 6500 50  0001 C CNN "LCSC"
 	1    5950 6500
 	1    0    0    -1
@@
 F 2 "Resistor_SMD:R_0603_1608Metric_Pad1.05x0.95mm_HandSolder" H 6500 6400 50  0001 C CNN
 F 3 "~" H 6500 6400 50  0001 C CNN
+F 4 "C22859" V 6500 6400 50  0001 C CNN "LCSC Part #"
 	1    6500 6400
 	0    1    1    0
@@
 F 2 "Resistor_SMD:R_0603_1608Metric_Pad1.05x0.95mm_HandSolder" H 6500 6600 50  0001 C CNN
 F 3 "~" H 6500 6600 50  0001 C CNN
+F 4 "C22859" V 6500 6600 50  0001 C CNN "LCSC"
 	1    6500 6600
 	0    1    1    0
@@
 F 2 "Diode_SMD:D_SMA" V 16050 2800 50  0001 C CNN
 F 3 "~" V 16050 2800 50  0001 C CNN
+F 4 "C110856" V 16050 2800 50  0001 C CNN "LCSC"
 	1    16050 2800
 	1    0    0    -1
@@
 F 2 "Speeduino_base:R0603" H 15850 7800 50  0001 C CNN
 F 3 "" H 15850 7800 50  0001 C CNN
+F 4 "C25803" H 15850 7800 50  0001 C CNN "LCSC"
 	1    15850 7800
 	1    0    0    -1
@@
 F 2 "Speeduino_base:R0603" H 15550 10200 50  0001 C CNN
 F 3 "~" H 15550 10200 50  0001 C CNN
+F 4 "C22775" V 15550 10200 50  0001 C CNN "LCSC"
 	1    15550 10200
 	0    1    1    0
@@
 F 2 "Speeduino_base:SOT23" H 12650 8050 50  0001 C CNN
 F 3 "" H 12650 8050 50  0001 C CNN
+F 4 "C19726" H 12650 8050 50  0001 C CNN "LCSC"
 	1    12650 8050
 	-1   0    0    -1
@@
 F 2 "Speeduino_base:SOT-23" H 14350 2200 50  0001 C CNN
 F 3 "" H 14350 2200 50  0001 C CNN
+F 4 "C344010" H 14350 2200 50  0001 C CNN "LCSC"
 	1    14350 2200
 	1    0    0    -1
@@
 F 2 "Speeduino_base:R0603" H 4650 10750 50  0001 C CNN
 F 3 "" H 4650 10750 50  0001 C CNN
+F 4 "C126158" H 4650 10750 50  0001 C CNN "LCSC"
 	1    4650 10750
 	0    -1   -1   0
@@
 F 2 "Speeduino_base:R0603" H 2950 11100 50  0001 C CNN
 F 3 "" H 2950 11100 50  0001 C CNN
+F 4 "C23186" H 2950 11100 50  0001 C CNN "LCSC"
 	1    2950 11100
 	0    -1   -1   0
@@
 F 2 "Speeduino_base:R0603" H 2750 10950 50  0001 C CNN
 F 3 "" H 2750 10950 50  0001 C CNN
+F 4 "C4216" H 2750 10950 50  0001 C CNN "LCSC"
 	1    2750 10950
 	-1   0    0    1
@@
 F 2 "Speeduino_base:C0603" H 1150 8000 50  0001 C CNN
 F 3 "" H 1150 8000 50  0001 C CNN
+F 4 "C21120" H 1150 8000 50  0001 C CNN "LCSC"
 	1    1150 8000
 	0    -1   -1   0
@@
 F 2 "Speeduino_base:R0603" H 950 7850 50  0001 C CNN
 F 3 "" H 950 7850 50  0001 C CNN
+F 4 "C23179" H 950 7850 50  0001 C CNN "LCSC"
 	1    950  7850
 	1    0    0    -1
@@
 F 2 "Speeduino_base:R0603" H 1550 8200 50  0001 C CNN
 F 3 "" H 1550 8200 50  0001 C CNN
+F 4 "C23260" H 1550 8200 50  0001 C CNN "LCSC"
 	1    1550 8200
 	1    0    0    -1
@@
 F 2 "Speeduino_base:R0603" H 1550 7850 50  0001 C CNN
 F 3 "" H 1550 7850 50  0001 C CNN
+F 4 "C23162" H 1550 7850 50  0001 C CNN "LCSC"
 	1    1550 7850
 	1    0    0    -1
@@
 Wire Wire Line
 	12750 7650 13200 7650
+$Comp
+L Speeduino_base-eagle-import:CERAMIC-10UF-25V-10%-X5R(1206) C15
+U 1 1 603F19F2
+P 3250 1090
+F 0 "C15" H 3100 1140 42  0000 L BNN
+F 1 "10uf" H 3100 990 42  0000 L BNN
+F 2 "Speeduino_base:C1206" H 3250 1090 50  0001 C CNN
+F 3 "" H 3250 1090 50  0001 C CNN
+F 4 "C13585" H 3250 1090 50  0001 C CNN "LCSC"
+	1    3250 1090
+	0    -1   -1   0
+$EndComp
+Wire Wire Line
+	3100 900  3250 900
+Wire Wire Line
+	3250 950  3250 940
+Connection ~ 3250 900
+Wire Wire Line
+	3250 900  3550 900
+Connection ~ 3250 940
+Wire Wire Line
+	3250 940  3250 900
 $EndSCHEMATC
